Commit message: Adding color to robotmodel

File: bme_ros2_project/urdf/mogi_bot.urdf (robot description, URDF)
Before this commit: robot mogi_bot, 10 links, 9 joints
Joints:
- joint camera_joint: origin xyz=0.225 0 0.075 rpy=0 0 0 -> xyz=0 -0.34875 0.10825 rpy=0 0 0
- joint scan_joint: origin xyz=0.0 0 0.15 rpy=0 0 0 -> xyz=0.0 0 0.42375 rpy=0 0 0

Commit message: Adding spawn_robot_launch.py

File: bme_ros2_project/urdf/mogi_bot.urdf (robot description, URDF)
Before this commit: robot mogi_bot, 10 links, 9 joints
Links:
- link base_link: geometry collision box size=.4 .7 .4; visual mesh filename=package://bme_ros2_project/meshes/mogi_bot.dae
- link front_left_wheel: geometry collision cylinder length=.08 radius=.095; visual mesh filename=package://bme_ros2_project/meshes/wheel.dae
- link front_right_wheel: geometry collision cylinder length=.08 radius=.095; visual mesh filename=package://bme_ros2_project/meshes/wheel.dae
- link rear_left_wheel: geometry collision cylinder length=.08 radius=.095; visual mesh filename=package://bme_ros2_project/meshes/wheel.dae
- link rear_right_wheel: geometry collision cylinder length=.08 radius=.095; visual mesh filename=package://bme_ros2_project/meshes/wheel.dae
Joints:
- joint imu_joint: origin xyz=0 0 0 rpy=0 0 0 -> xyz=0 0 0 rpy=0 0 -1.5707

Commit message: Correcting urdf file

File: bme_ros2_project/urdf/mogi_bot.urdf (robot description, URDF)
Before this commit: robot mogi_bot, 10 links, 9 joints
Links:
- link base_link: geometry collision box size=.7 .4 .4; visual mesh filename=package://bme_ros2_project/meshes/mogi_bot.dae
Joints:
- joint camera_joint: origin xyz=0 -0.34875 0.10825 rpy=0 0 0 -> xyz=0.34875 0 0.10825 rpy=0 0 0
- joint front_left_wheel_joint: axis 1 0 0 -> 0 1 0
- joint front_right_wheel_joint: axis 1 0 0 -> 0 1 0
- joint imu_joint: origin xyz=0 0 0 rpy=0 0 -1.5707 -> xyz=0 0 0 rpy=0 0 0
- joint rear_left_wheel_joint: axis 1 0 0 -> 0 1 0; origin xyz=-0.125 0.12875 0.0375 rpy=0 3.14159 0 -> xyz=-0.125 0.12875 0.0375 rpy=0 0 0
- joint rear_right_wheel_joint: axis 1 0 0 -> 0 1 0; origin xyz=-0.125 -0.12875 0.0375 rpy=0 3.14159 0 -> xyz=-0.125 -0.12875 0.0375 rpy=0 0 0
- joint scan_joint: axis 0 1 0 -> 1 0 0; origin xyz=0.0 0 0.42375 rpy=0 0 0 -> xyz=0.0 0 0.44375 rpy=0 0 0
